File: keyboard-pcb/keyboard-pcb.kicad_pcb (KiCad board)
At the start: 2 copper layers, 86.4 x 177.8 mm, 72 parts, among them J1 Conn_02x03_Odd_Even, SW1 SW_Push, SW10 SW_Push, SW11 SW_Push, SW12 SW_Push, SW13 SW_Push, SW14 SW_Push, SW15 SW_Push, SW16 SW_Push, SW17 SW_Push, SW18 SW_Push, SW19 SW_Push, SW2 SW_Push, SW20 SW_Push, SW21 SW_Push, SW22 SW_Push, SW23 SW_Push, SW24 SW_Push, SW25 SW_Push, SW26 SW_Push, SW27 SW_Push, SW28 SW_Push, SW3 SW_Push, SW4 SW_Push, SW5 SW_SPST, SW6 SW_Push, SW7 SW_Push, SW8 SW_Push, SW9 SW_Push, U1 R1500H, U2 ATmega328-P, U3 RC1602A

Commit message: Rev1 PCB as built; debugging keyboard software
Other:
- board text added: "UPCO Graphics Systems -- Programmer's Calculator -- V1.0 2024-03 -- E. Hazen"
Changed lines of the file:
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@@
   (gr_line (start 29.21 195.58) (end 29.21 17.78)
     (stroke (width 0.1) (type default)) (layer "Edge.Cuts"))
+  (gr_text "UPCO Graphics Systems -- Programmer's Calculator -- V1.0 2024-03 -- E. Hazen" (at 32.639 171.323 90) (layer "F.SilkS")
+    (effects (font (size 1.651 1.651) (thickness 0.2032)) (justify left bottom))
+  )
   (segment (start 38.735 58.42) (end 43.18 58.42) (width 0.254) (layer "B.Cu") (net 1))
   (segment (start 86.995 58.42) (end 83.82 58.42) (width 0.254) (layer "B.Cu") (net 2))
