File: keyboard-pcb/keyboard-pcb.kicad_sch (KiCad schematic)
At the start: 72 parts, among them J1 Conn_02x03_Odd_Even, SW1 SW_Push, SW10 SW_Push, SW11 SW_Push, SW12 SW_Push, SW13 SW_Push, SW14 SW_Push, SW15 SW_Push, SW16 SW_Push, SW17 SW_Push, SW18 SW_Push, SW19 SW_Push, SW2 SW_Push, SW20 SW_Push, SW21 SW_Push, SW22 SW_Push, SW23 SW_Push, SW24 SW_Push, SW25 SW_Push, SW26 SW_Push, SW27 SW_Push, SW28 SW_Push, SW3 SW_Push, SW4 SW_Push, SW5 SW_SPST, SW6 SW_Push, SW7 SW_Push, SW8 SW_Push, SW9 SW_Push, U1 R1500H, U2 ATmega328-P, U3 RC1602A

Commit message: Rev1 PCB as built; debugging keyboard software
Parts:
- renumbered U1 to U2, U2 to U3, U3 to U4
Changed lines of the file:
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@@
+    (stroke (width 0) (type default))
+  )
+  (wire (pts (xy 240.03 54.61) (xy 246.38 54.61))
     (stroke (width 0) (type default))
   )
@@
   )
   (wire (pts (xy 158.75 121.92) (xy 158.75 134.62))
-    (stroke (width 0) (type default))
-  )
-  (wire (pts (xy 240.03 54.61) (xy 246.38 54.61))
     (stroke (width 0) (type default))
   )
@@
   (symbol (lib_id "Display_Character:RC1602A") (at 49.53 165.1 0) (mirror y) (unit 1)
     (in_bom yes) (on_board yes) (dnp no)
-    (property "Reference" "U3" (at 47.5741 146.05 0)
+    (property "Reference" "U4" (at 47.5741 146.05 0)
       (effects (font (size 1.27 1.27)) (justify left))
     )
@@
       (project "keyboard-pcb"
         (path "/1f3a3fa9-d994-4670-aaa6-06c93cb2d887"
-          (reference "U3") (unit 1)
+          (reference "U4") (unit 1)
         )
       )
@@
   (symbol (lib_id "MCU_Microchip_ATmega:ATmega328-P") (at 45.72 67.31 0) (unit 1)
     (in_bom yes) (on_board yes) (dnp no)
-    (property "Reference" "U2" (at 36.83 64.77 0)
+    (property "Reference" "U3" (at 36.83 64.77 0)
       (effects (font (size 1.27 1.27)))
     )
@@
       (project "keyboard-pcb"
         (path "/1f3a3fa9-d994-4670-aaa6-06c93cb2d887"
-          (reference "U2") (unit 1)
+          (reference "U3") (unit 1)
         )
       )
@@
   (symbol (lib_id "power:VCC") (at 246.38 48.26 0) (mirror y) (unit 1)
     (in_bom yes) (on_board yes) (dnp no)
-    (property "Reference" "#PWR04" (at 246.38 52.07 0)
+    (property "Reference" "#PWR05" (at 246.38 52.07 0)
       (effects (font (size 1.27 1.27)) hide)
     )
@@
       (project "keyboard-pcb"
         (path "/1f3a3fa9-d994-4670-aaa6-06c93cb2d887"
-          (reference "#PWR04") (unit 1)
+          (reference "#PWR05") (unit 1)
         )
       )
@@
   (symbol (lib_id "power:VCC") (at 49.53 143.51 0) (unit 1)
     (in_bom yes) (on_board yes) (dnp no) (fields_autoplaced)
-    (property "Reference" "#PWR07" (at 49.53 147.32 0)
+    (property "Reference" "#PWR08" (at 49.53 147.32 0)
       (effects (font (size 1.27 1.27)) hide)
     )
@@
       (project "keyboard-pcb"
         (path "/1f3a3fa9-d994-4670-aaa6-06c93cb2d887"
-          (reference "#PWR07") (unit 1)
+          (reference "#PWR08") (unit 1)
         )
       )
@@
   (symbol (lib_id "R1500H_vreg:R1500H") (at 231.14 55.88 0) (unit 1)
     (in_bom yes) (on_board yes) (dnp no)
-    (property "Reference" "U1" (at 226.06 50.8 0)
+    (property "Reference" "U2" (at 226.06 50.8 0)
       (effects (font (size 1.27 1.27)))
     )
@@
       (project "keyboard-pcb"
         (path "/1f3a3fa9-d994-4670-aaa6-06c93cb2d887"
-          (reference "U1") (unit 1)
+          (reference "U2") (unit 1)
         )
       )
@@
   (symbol (lib_id "power:GND") (at 204.47 73.66 0) (mirror y) (unit 1)
     (in_bom yes) (on_board yes) (dnp no)
-    (property "Reference" "#PWR05" (at 204.47 80.01 0)
+    (property "Reference" "#PWR06" (at 204.47 80.01 0)
       (effects (font (size 1.27 1.27)) hide)
     )
@@
       (project "keyboard-pcb"
         (path "/1f3a3fa9-d994-4670-aaa6-06c93cb2d887"
-          (reference "#PWR05") (unit 1)
+          (reference "#PWR06") (unit 1)
         )
       )
@@
   (symbol (lib_id "power:GND") (at 45.72 107.95 0) (unit 1)
     (in_bom yes) (on_board yes) (dnp no) (fields_autoplaced)
-    (property "Reference" "#PWR06" (at 45.72 114.3 0)
+    (property "Reference" "#PWR07" (at 45.72 114.3 0)
       (effects (font (size 1.27 1.27)) hide)
     )
@@
       (project "keyboard-pcb"
         (path "/1f3a3fa9-d994-4670-aaa6-06c93cb2d887"
-          (reference "#PWR06") (unit 1)
+          (reference "#PWR07") (unit 1)
         )
       )
@@
   (symbol (lib_id "power:VCC") (at 118.11 161.29 0) (unit 1)
     (in_bom yes) (on_board yes) (dnp no) (fields_autoplaced)
-    (property "Reference" "#PWR09" (at 118.11 165.1 0)
+    (property "Reference" "#PWR010" (at 118.11 165.1 0)
       (effects (font (size 1.27 1.27)) hide)
     )
@@
       (project "keyboard-pcb"
         (path "/1f3a3fa9-d994-4670-aaa6-06c93cb2d887"
-          (reference "#PWR09") (unit 1)
+          (reference "#PWR010") (unit 1)
         )
       )
@@
   (symbol (lib_id "power:GND") (at 49.53 184.15 0) (unit 1)
     (in_bom yes) (on_board yes) (dnp no) (fields_autoplaced)
-    (property "Reference" "#PWR011" (at 49.53 190.5 0)
+    (property "Reference" "#PWR012" (at 49.53 190.5 0)
       (effects (font (size 1.27 1.27)) hide)
     )
@@
       (project "keyboard-pcb"
         (path "/1f3a3fa9-d994-4670-aaa6-06c93cb2d887"
-          (reference "#PWR011") (unit 1)
+          (reference "#PWR012") (unit 1)
         )
       )
@@
   (symbol (lib_id "power:VCC") (at 85.09 153.67 0) (unit 1)
     (in_bom yes) (on_board yes) (dnp no) (fields_autoplaced)
-    (property "Reference" "#PWR08" (at 85.09 157.48 0)
+    (property "Reference" "#PWR09" (at 85.09 157.48 0)
       (effects (font (size 1.27 1.27)) hide)
     )
@@
       (project "keyboard-pcb"
         (path "/1f3a3fa9-d994-4670-aaa6-06c93cb2d887"
-          (reference "#PWR08") (unit 1)
+          (reference "#PWR09") (unit 1)
         )
       )
@@
   (symbol (lib_id "power:GND") (at 118.11 172.72 0) (unit 1)
     (in_bom yes) (on_board yes) (dnp no) (fields_autoplaced)
-    (property "Reference" "#PWR010" (at 118.11 179.07 0)
+    (property "Reference" "#PWR011" (at 118.11 179.07 0)
       (effects (font (size 1.27 1.27)) hide)
     )
@@
       (project "keyboard-pcb"
         (path "/1f3a3fa9-d994-4670-aaa6-06c93cb2d887"
-          (reference "#PWR010") (unit 1)
-        )
-      )
+          (reference "#PWR011") (unit 1)
+        )
+      )
